File: Hardware/Production SKU/SparkFun_Bluetooth_Beacon_IN100.sch (EAGLE design)
At the start: 34 parts, among them J3 Vertical Qwiic Connector, U1 IN100, Y1 CRYSTAL-26MHZSMD-3.2X2.5

Commit message: Fix production SKU board and schematic being inconsistent
Parts:
- D1: value RED -> DNP
- R1: value 2.2k -> DNP
- RST: value MOMENTARY-SWITCH-SPST-SMD-4.6X2.8MM -> DNP
Changed lines of the file:
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@@
 <part name="LOGO1" library="SparkFun-Aesthetics" deviceset="OSHW-LOGO" device="S"/>
 <part name="LOGO2" library="SparkFun-Aesthetics" deviceset="SFE_LOGO_NAME_FLAME" device=".1_INCH"/>
-<part name="D1" library="SparkFun-LED" deviceset="LED-RED" device="_0402" value="RED">
+<part name="D1" library="SparkFun-LED" deviceset="LED-RED" device="_0402" value="DNP">
 <attribute name="PROD_ID" value=""/>
 </part>
-<part name="R1" library="SparkFun-Resistors" deviceset="2.2KOHM" device="-0402T-1/16W-1%" value="2.2k">
+<part name="R1" library="SparkFun-Resistors" deviceset="2.2KOHM" device="-0402T-1/16W-1%" value="DNP">
 <attribute name="PROD_ID" value=""/>
 </part>
@@
 <part name="SUPPLY1" library="SparkFun-PowerSymbols" deviceset="VCC" device=""/>
 <part name="SUPPLY5" library="SparkFun-PowerSymbols" deviceset="VCC" device=""/>
-<part name="RST" library="SparkFun-Switches" deviceset="MOMENTARY-SWITCH-SPST" device="-SMD-4.6X2.8MM">
+<part name="RST" library="SparkFun-Switches" deviceset="MOMENTARY-SWITCH-SPST" device="-SMD-4.6X2.8MM" value="DNP">
 <attribute name="PROD_ID" value=""/>
 </part>
