File: Hardware/NanoBeacon Lite/SparkFun NanoBeacon Lite Board - IN100.brd (EAGLE design)
At the start: 25.4 x 25.4 mm, 63 parts, among them J3 Vertical Qwiic Connector, U1 IN100, Y1 CRYSTAL-26MHZSMD-3.2X2.5

Commit message: Remove library file
Part is in SFE Eagle library, update part in design
Parts:
- E1: value ANTENNA-GROUNDEDTRACE-15.2MM -> ANTENNA-GROUNDEDTRACE-15.2MM-MIRROR; device SparkFun-RF:TRACE_ANTENNA_2.4GHZ_15.2MM -> SparkFun-RF:TRACE_ANTENNA_2.4GHZ_15.2MM_MIRROR
- U1: device IN100:IN100 -> SparkFun-RF:IN100
Changed lines of the file:
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@@
 </autorouter>
 <elements>
-<element name="E1" library="SparkFun-RF" package="TRACE_ANTENNA_2.4GHZ_15.2MM" value="ANTENNA-GROUNDEDTRACE-15.2MM" x="17.399" y="20.193" smashed="yes">
+<element name="E1" library="SparkFun-RF" package="TRACE_ANTENNA_2.4GHZ_15.2MM_MIRROR" value="ANTENNA-GROUNDEDTRACE-15.2MM-MIRROR" x="17.399" y="20.193" smashed="yes">
 <attribute name="NAME" x="17.399" y="21.463" size="0.6096" layer="25" font="vector" ratio="20" align="bottom-center"/>
 <attribute name="VALUE" x="17.399" y="21.209" size="0.6096" layer="27" font="vector" ratio="20" align="top-center"/>
@@
 <attribute name="REV" value="" x="-10.16" y="-25.4" size="1.778" layer="27" font="vector" ratio="15" display="off"/>
 </element>
-<element name="U1" library="IN100" package="IN100" value="IN100" x="12.7" y="15.875" smashed="yes">
+<element name="U1" library="SparkFun-RF" package="IN100" value="IN100" x="12.7" y="15.875" smashed="yes">
 <attribute name="NAME" x="12.7" y="18.125" size="0.6096" layer="25" font="vector" ratio="20" align="center"/>
 <attribute name="PROD_ID" value="IC-17260" x="12.7" y="15.875" size="1.778" layer="27" display="off"/>
@@
 <element name="BT1" library="SparkFun-Batteries" package="BATTCON_12MM" value="" x="12.7" y="6.985" smashed="yes" rot="R180">
 <attribute name="NAME" x="23.495" y="6.985" size="0.6096" layer="25" font="vector" ratio="20" rot="R270" align="bottom-center"/>
-<attribute name="PROD_ID" value="BATT-08044" x="12.7" y="6.985" size="1.778" layer="27" font="vector" ratio="15" rot="R180" display="off"/>
-<attribute name="SF_SKU" value="PRT-10592" x="12.7" y="6.985" size="1.778" layer="27" font="vector" ratio="15" rot="R180" display="off"/>
 <attribute name="VALUE" x="12.7" y="6.985" size="0.6096" layer="27" font="vector" ratio="20" rot="R270" align="top-center"/>
 </element>
@@
 <wire x1="22.7838" y1="11.4479875" x2="22.7838" y2="12.6238" width="0.4064" layer="1"/>
 <wire x1="22.7838" y1="12.6238" x2="24.13" y2="13.97" width="0.4064" layer="1"/>
-<contactref element="BT1" pad="PWR@2"/>
 <contactref element="D1" pad="A"/>
 <wire x1="4.826" y1="6.985" x2="5.58" y2="7.739" width="0.2032" layer="1"/>
@@
 <wire x1="6.48986875" y1="12.446" x2="6.485" y2="12.446" width="0.2032" layer="1"/>
 <wire x1="5.58" y1="10.16" x2="6.731" y2="10.16" width="0.2032" layer="1"/>
+<contactref element="BT1" pad="PWR@2"/>
 <wire x1="6.485" y1="12.446" x2="12.95" y2="17.275" width="0" layer="19" extent="1-1"/>
 </signal>
